Commit message: Testes para pratica 3

File: model_description/urdf/hot_wheels.urdf (robot description, URDF)
Before this commit: robot hot_wheels, 5 links, 4 joints
Links:
- link base_link: mass 1.9 -> 5.0
- link caster_link: mass 0.1 -> 0.5
- link left_wheel: mass 0.2 -> 1.0; geometry collision cylinder length=0.03 radius=0.05; visual cylinder length=0.03 radius=0.05
- link right_wheel: mass 0.2 -> 1.0; geometry collision cylinder length=0.03 radius=0.05; visual cylinder length=0.03 radius=0.05

Commit message: Minor Fixes

File: model_description/urdf/hot_wheels.urdf (robot description, URDF)
Before this commit: robot hot_wheels, 5 links, 4 joints
Links:
- added link camera_link, mass 0.005; visual box size=0.030 0.040 0.025
- added link camera_optical_frame
- added link gps_link, mass 0.005; visual cylinder length=0.012 radius=0.015
- added link imu_link, mass 0.005; visual box size=0.025 0.025 0.015
- added link lidar_link, mass 0.005; visual cylinder length=0.020 radius=0.025
Joints:
- added joint camera_joint: type fixed, parent base_link, child camera_link, origin xyz=0.120 0 0.020 rpy=0 0 0
- added joint camera_optical_joint: type fixed, parent camera_link, child camera_optical_frame, origin xyz=0.015 0 0 rpy=-1.57079632679 0 -1.57079632679
- added joint gps_joint: type fixed, parent base_link, child gps_link, origin xyz=-0.045 -0.037 0.060 rpy=0 0 0
- added joint imu_joint: type fixed, parent base_link, child imu_link, origin xyz=-0.045 0.037 0.060 rpy=0 0 0
- added joint lidar_joint: type fixed, parent base_link, child lidar_link, origin xyz=0.075 0 0.075 rpy=0 0 0
- joint left_wheel_joint: limit (none) -> effort=10000.0 velocity=10.0
- joint right_wheel_joint: limit (none) -> effort=10000.0 velocity=10.0
